Commit message: Update Boying calf joint torque limit from 60 to 90 N·m
FL/FR/RL/RR_calf_joint effort: 60 -> 90 N·m
Hip and thigh joints remain at 60 N·m

Co-Authored-By: Claude Code <noreply@anthropic.com>

File: resources/robots/boying_description/urdf/boying_description_withouthm.urdf (robot description, URDF)
Before this commit: robot boying, 19 links, 18 joints
Joints:
- joint FL_calf_joint: limit lower=-2.7478 upper=-0.9269 effort=60 velocity=10.4 -> lower=-2.7478 upper=-0.9269 effort=90 velocity=10.4
- joint FR_calf_joint: limit lower=-2.7478 upper=-0.9269 effort=60 velocity=10.4 -> lower=-2.7478 upper=-0.9269 effort=90 velocity=10.4
- joint RL_calf_joint: limit lower=-2.7478 upper=-0.9269 effort=60 velocity=10.4 -> lower=-2.7478 upper=-0.9269 effort=90 velocity=10.4
- joint RR_calf_joint: limit lower=-2.7478 upper=-0.9269 effort=60 velocity=10.4 -> lower=-2.7478 upper=-0.9269 effort=90 velocity=10.4

Commit message: Tune boying PD gains and default joint angles
- Kp: 60 → 50, Kd: 4.5 → 2.25
- thigh default angles: FL/FR 0.8→0.7, RL/RR 1.0→0.8
- Update all related comments to reflect new PD values
- URDF: expand collision geometry for thigh/calf/foot links

Co-Authored-By: Claude Opus 4.7 (1M context) <noreply@anthropic.com>

File: resources/robots/boying_description/urdf/boying_description_withouthm.urdf (robot description, URDF)
Before this commit: robot boying, 19 links, 18 joints
Links:
- link FL_calf: geometry collision cylinder length=0.22 radius=0.009; visual mesh filename=../meshes/L_calf.STL
- link FL_thigh: geometry collision box size=0.03 0.03 0.23; collision cylinder length=0.0700 radius=0.044
- link FR_calf: geometry collision cylinder length=0.22 radius=0.009; visual mesh filename=../meshes/R_calf.STL
- link FR_thigh: geometry collision box size=0.03 0.03 0.23; collision cylinder length=0.0700 radius=0.044
- link RL_calf: geometry collision cylinder length=0.22 radius=0.009; visual mesh filename=../meshes/L_calf.STL
- link RL_thigh: geometry collision box size=0.03 0.03 0.23; collision cylinder length=0.0700 radius=0.044
- link RR_calf: geometry collision cylinder length=0.22 radius=0.009; visual mesh filename=../meshes/R_calf.STL
- link RR_thigh: geometry collision box size=0.03 0.03 0.23; collision cylinder length=0.0700 radius=0.044
- link base: geometry collision box size=0.430 0.180 0.136; visual mesh filename=../meshes/base.STL
